File: crazyflie-usd-spi3.kicad_pcb (KiCad board)
At the start: 2 copper layers, 27 x 22 mm, 7 parts, among them J1 Left, J2 Right, J3 Left, J4 Right, J5 microSD, U1 DS28E05

Commit message: As sent to JLCPCB? but actually exported?
Parts:
- moved J1 0.50 mm to (138.5, 68.0)
- moved J2 0.50 mm to (160.5, 68.0)
- moved J3 0.50 mm to (138.5, 59.0)
- moved J4 0.50 mm to (160.5, 59.0)
Routing:
- net VCC: track 42.8 -> 48.2 mm, vias 4 -> 5
- net /IO4: track 22.4 -> 20.6 mm
- net /SCK3: track 18.0 -> 18.5 mm
- net /OW: track 17.9 -> 18.4 mm
- net /MISO3: track 20.3 -> 20.8 mm
Other:
- board size 27 x 22 mm -> 28 x 22 mm
- rule pad_to_mask_clearance: 0.051 -> 0.05
- rule solder_mask_min_width: 0.25 -> 0.15
- board text added: "FRONT DOWN"
