File: crazyflie-usd-spi3.sch (KiCad schematic (older format))
At the start: 7 parts, among them J1 Left, J2 Right, J3 Left, J4 Right, J5 microSD, U1 DS28E05

Commit message: As sent to JLCPCB? but actually exported?
Other:
- note added: "(connector used instead of symbol for DS28E05\nso as to not use any external libraries)"
- note added: "Two connector symbols for each side…\none for the through-holes, one for the SMD pads"
- note removed: "(connector used instead\nof symbol for DS28E05\nso as to not use any ext. libs.)"
- moved on the sheet: C1, J5
Changed lines of the file:
@@
 L Connector_Generic:Conn_01x10 J5
 U 1 1 5E7E354F
-P 6650 1850
-F 0 "J5" H 6650 2400 50  0000 C BNN
-F 1 "microSD" H 6650 2350 50  0000 C CNN
-F 2 "stdpads:Molex_473521001_microSD" H 6650 1850 50  0001 C CNN
-F 3 "~" H 6650 1850 50  0001 C CNN
-	1    6650 1850
-	1    0    0    -1
-$EndComp
-Text Notes 6150 2700 0    40   ~ 0
+P 5800 1850
+F 0 "J5" H 5800 2400 50  0000 C BNN
+F 1 "microSD" H 5800 2350 50  0000 C CNN
+F 2 "stdpads:Molex_473521001_microSD" H 5800 1850 50  0001 C CNN
+F 3 "~" H 5800 1850 50  0001 C CNN
+	1    5800 1850
+	1    0    0    -1
+$EndComp
+Text Notes 5300 2700 0    50   ~ 0
 Pinout is for Molex 473521001\nmicroSD connector
 $Comp
 L power:VCC #PWR0104
 U 1 1 5E7D8CF1
-P 6150 1750
-F 0 "#PWR0104" H 6150 1600 50  0001 C CNN
-F 1 "VCC" H 6150 1900 50  0000 C CNN
-F 2 "" H 6150 1750 50  0001 C CNN
-F 3 "" H 6150 1750 50  0001 C CNN
-	1    6150 1750
-	1    0    0    -1
-$EndComp
-Text Label 6250 1850 0    50   ~ 0
+P 5300 1750
+F 0 "#PWR0104" H 5300 1600 50  0001 C CNN
+F 1 "VCC" H 5300 1900 50  0000 C CNN
+F 2 "" H 5300 1750 50  0001 C CNN
+F 3 "" H 5300 1750 50  0001 C CNN
+	1    5300 1750
+	1    0    0    -1
+$EndComp
+Text Label 5400 1850 0    50   ~ 0
 SCK3
 Wire Wire Line
-	6250 1850 6450 1850
+	5400 1850 5600 1850
 $Comp
 L power:GND #PWR0105
 U 1 1 5E7DA291
-P 6150 1950
-F 0 "#PWR0105" H 6150 1700 50  0001 C CNN
-F 1 "GND" H 6150 1800 50  0000 C CNN
-F 2 "" H 6150 1950 50  0001 C CNN
-F 3 "" H 6150 1950 50  0001 C CNN
-	1    6150 1950
-	1    0    0    -1
-$EndComp
-Wire Wire Line
-	6150 1950 6450 1950
-Text Label 6250 2050 0    50   ~ 0
+P 5300 1950
+F 0 "#PWR0105" H 5300 1700 50  0001 C CNN
+F 1 "GND" H 5300 1800 50  0000 C CNN
+F 2 "" H 5300 1950 50  0001 C CNN
+F 3 "" H 5300 1950 50  0001 C CNN
+	1    5300 1950
+	1    0    0    -1
+$EndComp
+Wire Wire Line
+	5300 1950 5600 1950
+Text Label 5400 2050 0    50   ~ 0
 MISO3
-Text Label 6250 1650 0    50   ~ 0
+Text Label 5400 1650 0    50   ~ 0
 MOSI3
-Text Label 6250 1550 0    50   ~ 0
+Text Label 5400 1550 0    50   ~ 0
 ~CS~3
 Wire Wire Line
-	6250 1550 6450 1550
-Wire Wire Line
-	6250 2050 6450 2050
-Wire Wire Line
-	6250 1650 6450 1650
-Wire Wire Line
-	6150 1750 6450 1750
+	5400 1550 5600 1550
+Wire Wire Line
+	5400 2050 5600 2050
+Wire Wire Line
+	5400 1650 5600 1650
+Wire Wire Line
+	5300 1750 5600 1750
 $Comp
 L power:GND #PWR0106
 U 1 1 5E7DD282
-P 6450 2350
-F 0 "#PWR0106" H 6450 2100 50  0001 C CNN
-F 1 "GND" H 6450 2200 50  0000 C CNN
-F 2 "" H 6450 2350 50  0001 C CNN
-F 3 "" H 6450 2350 50  0001 C CNN
-	1    6450 2350
-	1    0    0    -1
-$EndComp
-Text Label 6250 2250 0    50   ~ 0
+P 5600 2350
+F 0 "#PWR0106" H 5600 2100 50  0001 C CNN
+F 1 "GND" H 5600 2200 50  0000 C CNN
+F 2 "" H 5600 2350 50  0001 C CNN
+F 3 "" H 5600 2350 50  0001 C CNN
+	1    5600 2350
+	1    0    0    -1
+$EndComp
+Text Label 5400 2250 0    50   ~ 0
 Detect
 Wire Wire Line
-	6250 2250 6450 2250
-Text Label 6250 2150 0    50   ~ 0
+	5400 2250 5600 2250
+Text Label 5400 2150 0    50   ~ 0
 SDD1
 Wire Wire Line
-	6250 2150 6450 2150
-Text Label 6250 1450 0    50   ~ 0
+	5400 2150 5600 2150
+Text Label 5400 1450 0    50   ~ 0
 SDD2
 Wire Wire Line
-	6250 1450 6450 1450
+	5400 1450 5600 1450
 $Comp
 L Device:C_Small C1
 U 1 1 5E7E357E
-P 7000 1900
-F 0 "C1" H 7092 1946 50  0000 L CNN
-F 1 "2u2" H 7092 1855 50  0000 L CNN
-F 2 "stdpads:C_0805" H 7000 1900 50  0001 C CNN
-F 3 "~" H 7000 1900 50  0001 C CNN
-	1    7000 1900
+P 6150 1900
+F 0 "C1" H 6242 1946 50  0000 L CNN
+F 1 "2u2" H 6242 1855 50  0000 L CNN
+F 2 "stdpads:C_0805" H 6150 1900 50  0001 C CNN
+F 3 "~" H 6150 1900 50  0001 C CNN
+	1    6150 1900
 	1    0    0    -1
 $EndComp
@@
 L power:GND #PWR0107
 U 1 1 5E7E41D4
-P 7000 2000
-F 0 "#PWR0107" H 7000 1750 50  0001 C CNN
-F 1 "GND" H 7000 1850 50  0000 C CNN
-F 2 "" H 7000 2000 50  0001 C CNN
-F 3 "" H 7000 2000 50  0001 C CNN
-	1    7000 2000
+P 6150 2000
+F 0 "#PWR0107" H 6150 1750 50  0001 C CNN
+F 1 "GND" H 6150 1850 50  0000 C CNN
+F 2 "" H 6150 2000 50  0001 C CNN
+F 3 "" H 6150 2000 50  0001 C CNN
+	1    6150 2000
 	1    0    0    -1
 $EndComp
@@
 L power:VCC #PWR0108
 U 1 1 5E7E4705
-P 7000 1800
-F 0 "#PWR0108" H 7000 1650 50  0001 C CNN
-F 1 "VCC" H 7000 1950 50  0000 C CNN
-F 2 "" H 7000 1800 50  0001 C CNN
-F 3 "" H 7000 1800 50  0001 C CNN
-	1    7000 1800
-	1    0    0    -1
-$EndComp
-Text Notes 3250 3000 0    40   ~ 0
+P 6150 1800
+F 0 "#PWR0108" H 6150 1650 50  0001 C CNN
+F 1 "VCC" H 6150 1950 50  0000 C CNN
+F 2 "" H 6150 1800 50  0001 C CNN
+F 3 "" H 6150 1800 50  0001 C CNN
+	1    6150 1800
+	1    0    0    -1
+$EndComp
+Text Notes 3250 2750 0    50   ~ 0
 DS28E05 implements\n1-wire serial deck identification
-Text Notes 3250 2800 0    40   ~ 0
-(connector used instead\nof symbol for DS28E05\nso as to not use any ext. libs.)
+Text Notes 3250 2950 0    50   ~ 0
+(connector used instead of symbol for DS28E05\nso as to not use any external libraries)
 $Comp
 L Connector_Generic:Conn_01x10 J3
@@
 Wire Wire Line
 	4300 2150 4500 2150
+Text Notes 2050 1200 0    50   ~ 0
+Two connector symbols for each side…\none for the through-holes, one for the SMD pads
 $EndSCHEMATC
